Commit message: modified for a demo - .xml & urdf combined in the fr5_cobot.py - demo_controller_FR5.py initialize

File: robopal/assets/models/manipulators/FR5Cobot/FR5Cobot.urdf (robot description, URDF)
Before this commit: robot fr5v6, 8 links, 7 joints
Links:
- link base_link: geometry collision mesh filename=package://frcobot_description/meshes/FR5Cobot/collision/bas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; visual mesh filename=package://frcobot_description/meshes/FR5Cobot/visual-stl/ba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
- link j1_Link: geometry collision mesh filename=package://frcobot_description/meshes/FR5Cobot/collision/j1_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; visual mesh filename=package://frcobot_description/meshes/FR5Cobot/visual-stl/j1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
- link j2_Link: geometry collision mesh filename=package://frcobot_description/meshes/FR5Cobot/collision/j2_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; visual mesh filename=package://frcobot_description/meshes/FR5Cobot/visual-stl/j2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
- link j3_Link: geometry collision mesh filename=package://frcobot_description/meshes/FR5Cobot/collision/j3_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; visual mesh filename=package://frcobot_description/meshes/FR5Cobot/visual-stl/j3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
- link j4_Link: geometry collision mesh filename=package://frcobot_description/meshes/FR5Cobot/collision/j4_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; visual mesh filename=package://frcobot_description/meshes/FR5Cobot/visual-stl/j4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
- link j5_Link: geometry collision mesh filename=package://frcobot_description/meshes/FR5Cobot/collision/j5_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; visual mesh filename=package://frcobot_description/meshes/FR5Cobot/visual-stl/j5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
- link j6_Link: geometry collision mesh filename=package://frcobot_description/meshes/FR5Cobot/collision/j6_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; visual mesh filename=package://frcobot_description/meshes/FR5Cobot/visual-stl/j6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

Commit message: manually set up the tool axis

File: robopal/assets/models/manipulators/FR5Cobot/FR5Cobot.urdf (robot description, URDF)
Before this commit: robot FR5Cobot, 8 links, 7 joints
Links:
- link base_link: geometry collision mesh filename=package://frcobot_description/meshes/FR5Cobot/collision/bas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; visual mesh filename=package://frcobot_description/meshes/FR5Cobot/visual/base_l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
- link j1_Link: geometry collision mesh filename=package://frcobot_description/meshes/FR5Cobot/collision/j1_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; visual mesh filename=package://frcobot_description/meshes/FR5Cobot/visual/j1_Lin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
- link j2_Link: geometry collision mesh filename=package://frcobot_description/meshes/FR5Cobot/collision/j2_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; visual mesh filename=package://frcobot_description/meshes/FR5Cobot/visual/j2_Lin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
- link j3_Link: geometry collision mesh filename=package://frcobot_description/meshes/FR5Cobot/collision/j3_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; visual mesh filename=package://frcobot_description/meshes/FR5Cobot/visual/j3_Lin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
- link j4_Link: geometry collision mesh filename=package://frcobot_description/meshes/FR5Cobot/collision/j4_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; visual mesh filename=package://frcobot_description/meshes/FR5Cobot/visual/j4_Lin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
- link j5_Link: geometry collision mesh filename=package://frcobot_description/meshes/FR5Cobot/collision/j5_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; visual mesh filename=package://frcobot_description/meshes/FR5Cobot/visual/j5_Lin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
- link j6_Link: geometry collision mesh filename=package://frcobot_description/meshes/FR5Cobot/collision/j6_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; visual mesh filename=package://frcobot_description/meshes/FR5Cobot/visual/j6_Lin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
Joints:
- joint j6: origin xyz=0 0 0.102 rpy=-1.5708 0 0 -> xyz=0 0.1 0.102 rpy=-1.5708 0 0
